Commit message: camera added to urdf file

File: urdf/model.urdf (robot description, URDF)
Before this commit: robot BLUE, 5 links, 4 joints
Links:
- removed link laser
- added link camera_link; collision cylinder length=0.05 radius=0.05; visual cylinder length=0.05 radius=0.05
Joints:
- removed joint base_to_hokuyo
- added joint base_to_camera: type fixed, parent base_link, child camera_link, origin xyz=1.05 0.0 0.187 rpy=0.0 0.15 0.0

Commit message: Camera added to launch and urdf files

File: urdf/model.urdf (robot description, URDF)
Before this commit: robot BLUE, 5 links, 4 joints
Joints:
- joint base_to_camera: origin xyz=1.05 0.0 0.187 rpy=0.0 0.15 0.0 -> xyz=0.455 -0.02 0.68 rpy=-0.02 0.0 0.06

Commit message: name of camera link changed, now we need a dynamic tf to attach this link with the real camera link

File: urdf/model.urdf (robot description, URDF)
Before this commit: robot BLUE, 5 links, 4 joints
Links:
- removed link camera_link
- added link camera_link_static; collision cylinder length=0.05 radius=0.05; visual cylinder length=0.05 radius=0.05
Joints:
- joint base_to_camera: child camera_link -> camera_link_static
