Commit message: New urdf model added for rviz representation

File: urdf/blue.urdf.xacro (robot description, xacro)
@@ -8,23 +8,20 @@
     <color rgba="0.5 0.5 0.5 1.0"/>
    </material>
+      <material name="white">
+    <color rgba="1.0 1.0 1.0 1.0"/>
+   </material>
    <material name="flat_black">
     <color rgba="0 0 0 1"/>
    </material>
-   <link name="world" />
    <link name="base_link"/>
-  <joint name="world_joint" type="fixed">
-    <parent link="world" />
-    <child link="base_link" />
-    <origin xyz="0.0 0.0 0.0" rpy="0.0 0.0 1.57" />
-  </joint>
   <joint name="blue_joint" type="fixed">
-    <parent link="world" />
+    <parent link="base_link" />
     <child link = "blue" />
-    <origin xyz="-0.4 -1.22 -0.435" rpy="1.57 0 1.57" />
+    <origin xyz="1.22 -0.4 -0.435" rpy="1.57 0 3.14" />
   </joint>
   <link name="blue">
     <visual>
       <geometry>
-        <mesh filename="package://blue_robot/meshes/base_alero.stl" scale="0.001 0.001 0.001"/>
+        <mesh filename="package://robot_blue/urdf/meshes/base_alero.stl" scale="0.001 0.001 0.001"/>
       </geometry>
       <material name="blue"/>
@@ -32,5 +29,5 @@
     <collision>
       <geometry>
-        <mesh filename="package://blue_robot/meshes/base_alero.stl" scale="0.001 0.001 0.001"/>
+        <mesh filename="package://robot_blue/urdf/meshes/base_alero.stl" scale="0.001 0.001 0.001"/>
       </geometry>
     </collision>
@@ -43,18 +40,42 @@
   </link>
   <joint name="velodyne_joint" type="fixed">
+    <parent link="base_link"/>
+    <child link="velodyne"/>
+    <origin rpy="0.0 0.0 0.0" xyz="0.55 0.0 0.645"/>
+  </joint>
+  <link name="velodyne"/>
+  <joint name="gps_joint" type="fixed">
+    <parent link="base_link"/>
+    <child link="gps"/>
+    <origin xyz="0.82 -0.25 0.0" rpy="0.0 0.0 0.0"/>
+  </joint>
+  <link name='gps'>
+    <visual>
+      <geometry>
+        <cylinder length="0.05" radius="0.07"/>
+      </geometry>
+      <material name="white"/>
+    </visual>
+    <collision>
+      <geometry>
+        <cylinder length="0.05" radius="0.07"/>
+      </geometry>
+    </collision>
+  </link>
+  <joint name="velodyne_visual_joint" type="fixed">
     <parent link="blue" />
-    <child link = "velodyne" />
+    <child link = "velodyne_visual" />
     <origin xyz="-0.1 0 0.4" rpy="-1.57 0 0" />
   </joint>
-  <link name="velodyne">
-    <visual>
-      <geometry>
-        <mesh filename="package://blue_robot/meshes/velodyne.stl" scale="0.001 0.001 0.001"/>
-      </geometry>
-      <material name="gray"/>
-    </visual>
-    <collision>
-      <geometry>
-        <mesh filename="package://blue_robot/meshes/velodyne.stl" scale="0.001 0.001 0.001"/>
+  <link name="velodyne_visual">
+    <visual>
+      <geometry>
+        <mesh filename="package://robot_blue/urdf/meshes/velodyne.stl" scale="0.001 0.001 0.001"/>
+      </geometry>
+      <material name="gray"/>
+    </visual>
+    <collision>
+      <geometry>
+        <mesh filename="package://robot_blue/urdf/meshes/velodyne.stl" scale="0.001 0.001 0.001"/>
       </geometry>
     </collision>
@@ -74,11 +95,11 @@
     <visual>
       <geometry>
-        <mesh filename="package://blue_robot/meshes/eje_delantero.stl" scale="0.001 0.001 0.001"/>
-      </geometry>
-      <material name="gray"/>
-    </visual>
-    <collision>
-      <geometry>
-        <mesh filename="package://blue_robot/meshes/eje_delantero.stl" scale="0.001 0.001 0.001"/>
+        <mesh filename="package://robot_blue/urdf/meshes/eje_delantero.stl" scale="0.001 0.001 0.001"/>
+      </geometry>
+      <material name="gray"/>
+    </visual>
+    <collision>
+      <geometry>
+        <mesh filename="package://robot_blue/urdf/meshes/eje_delantero.stl" scale="0.001 0.001 0.001"/>
       </geometry>
     </collision>
@@ -98,5 +119,5 @@
     <visual>
       <geometry>
-        <mesh filename="package://blue_robot/meshes/rueda_d.stl" scale="0.001 0.001 0.001"/>
+        <mesh filename="package://robot_blue/urdf/meshes/rueda_d.stl" scale="0.001 0.001 0.001"/>
       </geometry>
       <material name="flat_black"/>
@@ -104,5 +125,5 @@
     <collision>
       <geometry>
-        <mesh filename="package://blue_robot/meshes/rueda_d.stl" scale="0.001 0.001 0.001"/>
+        <mesh filename="package://robot_blue/urdf/meshes/rueda_d.stl" scale="0.001 0.001 0.001"/>
       </geometry>
     </collision>
@@ -122,11 +143,11 @@
     <visual>
       <geometry>
-        <mesh filename="package://blue_robot/meshes/aro_delantero.stl" scale="0.001 0.001 0.001"/>
-      </geometry>
-      <material name="gray"/>
-    </visual>
-    <collision>
-      <geometry>
-        <mesh filename="package://blue_robot/meshes/aro_delantero.stl" scale="0.001 0.001 0.001"/>
+        <mesh filename="package://robot_blue/urdf/meshes/aro_delantero.stl" scale="0.001 0.001 0.001"/>
+      </geometry>
+      <material name="gray"/>
+    </visual>
+    <collision>
+      <geometry>
+        <mesh filename="package://robot_blue/urdf/meshes/aro_delantero.stl" scale="0.001 0.001 0.001"/>
       </geometry>
     </collision>
@@ -146,5 +167,5 @@
     <visual>
       <geometry>
-        <mesh filename="package://blue_robot/meshes/rueda_i.stl" scale="0.001 0.001 0.001"/>
+        <mesh filename="package://robot_blue/urdf/meshes/rueda_i.stl" scale="0.001 0.001 0.001"/>
       </geometry>
       <material name="flat_black"/>
@@ -152,5 +173,5 @@
     <collision>
       <geometry>
-        <mesh filename="package://blue_robot/meshes/rueda_i.stl" scale="0.001 0.001 0.001"/>
+        <mesh filename="package://robot_blue/urdf/meshes/rueda_i.stl" scale="0.001 0.001 0.001"/>
       </geometry>
     </collision>
@@ -170,11 +191,11 @@
     <visual>
       <geometry>
-        <mesh filename="package://blue_robot/meshes/aro_delantero.stl" scale="0.001 0.001 0.001"/>
-      </geometry>
-      <material name="gray"/>
-    </visual>
-    <collision>
-      <geometry>
-        <mesh filename="package://blue_robot/meshes/aro_delantero.stl" scale="0.001 0.001 0.001"/>
+        <mesh filename="package://robot_blue/urdf/meshes/aro_delantero.stl" scale="0.001 0.001 0.001"/>
+      </geometry>
+      <material name="gray"/>
+    </visual>
+    <collision>
+      <geometry>
+        <mesh filename="package://robot_blue/urdf/meshes/aro_delantero.stl" scale="0.001 0.001 0.001"/>
       </geometry>
     </collision>
@@ -194,11 +215,11 @@
     <visual>
       <geometry>
-        <mesh filename="package://blue_robot/meshes/eje_trasero.stl" scale="0.001 0.001 0.001"/>
-      </geometry>
-      <material name="gray"/>
-    </visual>
-    <collision>
-      <geometry>
-        <mesh filename="package://blue_robot/meshes/eje_trasero.stl" scale="0.001 0.001 0.001"/>
+        <mesh filename="package://robot_blue/urdf/meshes/eje_trasero.stl" scale="0.001 0.001 0.001"/>
+      </geometry>
+      <material name="gray"/>
+    </visual>
+    <collision>
+      <geometry>
+        <mesh filename="package://robot_blue/urdf/meshes/eje_trasero.stl" scale="0.001 0.001 0.001"/>
       </geometry>
     </collision>
@@ -218,5 +239,5 @@
     <visual>
       <geometry>
-        <mesh filename="package://blue_robot/meshes/rueda_trasera.stl" scale="0.001 0.001 0.001"/>
+        <mesh filename="package://robot_blue/urdf/meshes/rueda_trasera.stl" scale="0.001 0.001 0.001"/>
       </geometry>
       <material name="flat_black"/>
@@ -224,5 +245,5 @@
     <collision>
       <geometry>
-        <mesh filename="package://blue_robot/meshes/rueda_trasera.stl" scale="0.001 0.001 0.001"/>
+        <mesh filename="package://robot_blue/urdf/meshes/rueda_trasera.stl" scale="0.001 0.001 0.001"/>
       </geometry>
     </collision>

Commit message: Lidar frame changed from velodyne to os_sensor.

File: urdf/blue.urdf.xacro (robot description, xacro)
@@ -39,10 +39,10 @@
     </inertial>
   </link>
-  <joint name="velodyne_joint" type="fixed">
+  <joint name="os_sensor_joint" type="fixed">
     <parent link="base_link"/>
-    <child link="velodyne"/>
+    <child link="os_sensor"/>
     <origin rpy="0.0 0.0 0.0" xyz="0.55 0.0 0.645"/>
   </joint>
-  <link name="velodyne"/>
+  <link name="os_sensor"/>
   <joint name="gps_joint" type="fixed">
     <parent link="base_link"/>
@@ -63,10 +63,10 @@
     </collision>
   </link>
-  <joint name="velodyne_visual_joint" type="fixed">
+  <joint name="os_sensor_visual_joint" type="fixed">
     <parent link="blue" />
-    <child link = "velodyne_visual" />
+    <child link = "os_sensor_visual" />
     <origin xyz="-0.1 0 0.4" rpy="-1.57 0 0" />
   </joint>
-  <link name="velodyne_visual">
+  <link name="os_sensor_visual">
     <visual>
       <geometry>
