Commit message: Gps position modified in urdf file.

File: robot_blue/urdf/blue.urdf.xacro (robot description, xacro)
@@ -48,5 +48,5 @@
     <parent link="base_link"/>
     <child link="gps"/>
-    <origin xyz="0.82 -0.25 0.0" rpy="0.0 0.0 0.0"/>
+    <origin xyz="0.0 -0.25 0.0" rpy="0.0 0.0 0.0"/>
   </joint>
   <link name='gps'>
