Commit message: Migration to ROS2, only start_tf launch file

File: robot_blue/urdf/blue.urdf.xacro (robot description, xacro)
@@ -39,10 +39,4 @@
     </inertial>
   </link>
-  <joint name="os_sensor_joint" type="fixed">
-    <parent link="base_link"/>
-    <child link="os_sensor"/>
-    <origin rpy="0.0 0.0 0.0" xyz="0.55 0.0 0.645"/>
-  </joint>
-  <link name="os_sensor"/>
   <joint name="gps_joint" type="fixed">
     <parent link="base_link"/>

Commit message: Fix tf tree

File: robot_blue/urdf/blue.urdf.xacro (robot description, xacro)
@@ -57,4 +57,10 @@
     </collision>
   </link>
+  <joint name="os_sensor_joint" type="fixed">
+    <parent link="base_link"/>
+    <child link="os_sensor"/>
+    <origin rpy="0.0 0.0 0.0" xyz="0.55 0.0 0.645"/>
+  </joint>
+  <link name="os_sensor"/>
   <joint name="os_sensor_visual_joint" type="fixed">
     <parent link="blue" />
